File: hardware/dronemagnav/sensors.kicad_sch (KiCad schematic)
At the start: 9 parts, among them U2 BMI088, U3 LIS3MDL, U4 BMP280

Commit message: Remove leftover ATC RoIP branding from the schematic title blocks
The sheet generator was copied from the other project and still stamped
the ATC RoIP company name into the title block of the five sub-sheets, so
it appeared on every schematic page and in Appendix A of the design
document. The title block now reads DroneMagNav Project, and the netlist
source path is project-relative. Schematic PDF and design document
regenerated; ERC unchanged (0 errors, 1 expected BMI088 warning).

Co-Authored-By: Claude Opus 5 <noreply@anthropic.com>
Other:
- company: ATC RoIP Gateway Project -> DroneMagNav Project
Changed lines of the file:
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@@
-(kicad_sch (version 20231120) (generator "atc_roip_gen")
+(kicad_sch (version 20231120) (generator "dronemagnav_gen")
   (paper "A3")
   (title_block
     (title "Sensors - BMI088 IMU, LIS3MDL magnetometer, BMP280 baro")
-    (company "ATC RoIP Gateway Project")
+    (company "DroneMagNav Project")
     (rev "A")
   )
